File: KickerBoard/KickerBoard.sch (EAGLE design)
At the start: 125 parts, among them IC1 MAX3051ESA+, IC2 TPD4S014DSQR, J1 SM03B-ZESS-TB, J2 J_USB_MICROAB_HIROSE_ZX62-AB-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, Q1 TK12P60W, Q4 BSS138, Q5 BSP130, Q6 ZXTN08400BFF, U1 LPC1549JBD48, U10 AD8601, U11 ADCMP350YKSZ, U12 MIC5219-3.3YMM, U2 LM5160QPWPRQ1, U3 UCC27212DPRT, U4 UCC27512DRSR, U5 IC-AD_ADR5041, U7 LT6108-2, U8 UCC27524DGN-NOPAD, U9 INA213, Y1 FA238V

Commit message: [fix] Kickerのコネクタのアサインを変更
Parts:
- added D12: (no value), MotorDriver:MOTORDRIVER_SBD-SOD523
- D1: value SMAJ60 -> SMAJ54A
- F1: value 10 -> 15
Connections:
- removed net CANH: IC1.CANH, J1.1
- removed net CANL: IC1.CANL, J1.2
- new net N$55: IC1.CANL, J1.3
- new net N$57: IC1.CANH, J1.2
- new net N$58: D12.A, J1.1
- net !RST: now also D12.K
- net GND: no longer J1.3
Other:
- note added: "自動放電回路"
- moved on the sheet: J1
Changed lines of the file:
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@@
 <?xml version="1.0" encoding="utf-8"?>
 <!DOCTYPE eagle SYSTEM "eagle.dtd">
-<eagle version="8.6.3">
+<eagle version="8.7.1">
 <drawing>
 <settings>
@@
 <part name="C10" library="Passive" deviceset="C" device="2012" value="0.1u"/>
 <part name="GND3" library="supply1" deviceset="GND" device=""/>
-<part name="F1" library="Passive" deviceset="F" device="3216" value="10"/>
+<part name="F1" library="Passive" deviceset="F" device="3216" value="15"/>
 <part name="+P2" library="supply1" deviceset="VBAT" device=""/>
 <part name="C5" library="Passive" deviceset="CPOL" device="S-6.3" value="22u"/>
-<part name="D1" library="Diode" deviceset="ZENER-*" device="DO-214AC" value="SMAJ60"/>
+<part name="D1" library="Diode" deviceset="ZENER-*" device="DO-214AC" value="SMAJ54A"/>
 <part name="GND4" library="supply1" deviceset="GND" device=""/>
 <part name="GND5" library="supply1" deviceset="GND" device=""/>
@@
 <part name="GND42" library="supply1" deviceset="GND" device=""/>
 <part name="J1" library="SM03B-ZESS-TB" library_urn="urn:adsk.eagle:library:1340468" deviceset="SM03B-ZESS-TB" device="" package3d_urn="urn:adsk.eagle:package:1340471/3"/>
-<part name="GND43" library="supply1" deviceset="GND" device=""/>
 <part name="U12" library="MIC5219-3.3YMM" deviceset="MIC5219-3.3YMM" device=""/>
 <part name="GND7" library="supply1" deviceset="GND" device=""/>
@@
 <part name="R52" library="MotorDriver" library_urn="urn:adsk.eagle:library:1073580" deviceset="R" device="1608" package3d_urn="urn:adsk.eagle:package:1073656/2" value="2.2"/>
 <part name="R53" library="MotorDriver" library_urn="urn:adsk.eagle:library:1073580" deviceset="R" device="1608" package3d_urn="urn:adsk.eagle:package:1073656/2" value="2.2"/>
+<part name="D12" library="MotorDriver" deviceset="MOTORDRIVER_SBD-*" device="SOD523"/>
 </parts>
 <sheets>
@@
 <instance part="GND41" gate="1" x="144.78" y="58.42"/>
 <instance part="GND42" gate="1" x="149.86" y="58.42"/>
-<instance part="J1" gate="G$1" x="160.02" y="78.74"/>
-<instance part="GND43" gate="1" x="154.94" y="58.42"/>
+<instance part="J1" gate="G$1" x="160.02" y="81.28"/>
 <instance part="J2" gate="G$1" x="177.8" y="-63.5"/>
 <instance part="J2" gate="G$2" x="177.8" y="-53.34"/>
@@
 <instance part="R48" gate="G$1" x="60.96" y="-15.24" rot="R180"/>
 <instance part="R49" gate="G$1" x="78.74" y="-40.64" rot="R90"/>
+<instance part="D12" gate="G$1" x="157.48" y="86.36" rot="R90"/>
 </instances>
 <busses>
@@
 </segment>
 <segment>
-<pinref part="J1" gate="G$1" pin="3"/>
-<wire x1="160.02" y1="73.66" x2="154.94" y2="73.66" width="0.1524" layer="91"/>
-<wire x1="154.94" y1="73.66" x2="154.94" y2="60.96" width="0.1524" layer="91"/>
-<pinref part="GND43" gate="1" pin="GND"/>
-</segment>
-<segment>
 <pinref part="J2" gate="G$1" pin="S4"/>
 <wire x1="182.88" y1="-66.04" x2="182.88" y2="-68.58" width="0.1524" layer="91"/>
@@
 <junction x="101.6" y="114.3"/>
 </segment>
+<segment>
+<pinref part="D12" gate="G$1" pin="K"/>
+<wire x1="157.48" y1="88.9" x2="157.48" y2="93.98" width="0.1524" layer="91"/>
+<label x="157.48" y="91.44" size="1.778" layer="95" rot="R90"/>
+</segment>
 </net>
 <net name="GATE_BUCK_L" class="0">
@@
 </segment>
 </net>
-<net name="CANH" class="0">
-<segment>
-<pinref part="IC1" gate="G$1" pin="CANH"/>
-<wire x1="142.24" y1="78.74" x2="160.02" y2="78.74" width="0.1524" layer="91"/>
-<label x="152.4" y="78.74" size="1.778" layer="95"/>
-<pinref part="J1" gate="G$1" pin="1"/>
-</segment>
-</net>
-<net name="CANL" class="0">
-<segment>
-<pinref part="IC1" gate="G$1" pin="CANL"/>
-<wire x1="142.24" y1="76.2" x2="160.02" y2="76.2" width="0.1524" layer="91"/>
-<label x="152.4" y="76.2" size="1.778" layer="95"/>
-<pinref part="J1" gate="G$1" pin="2"/>
-</segment>
-</net>
 <net name="ID" class="0">
 <segment>
@@
 <wire x1="78.74" y1="-45.72" x2="78.74" y2="-50.8" width="0.1524" layer="91"/>
 <wire x1="78.74" y1="-50.8" x2="83.82" y2="-50.8" width="0.1524" layer="91"/>
+</segment>
+</net>
+<net name="N$55" class="0">
+<segment>
+<pinref part="IC1" gate="G$1" pin="CANL"/>
+<pinref part="J1" gate="G$1" pin="3"/>
+<wire x1="142.24" y1="76.2" x2="160.02" y2="76.2" width="0.1524" layer="91"/>
+</segment>
+</net>
+<net name="N$57" class="0">
+<segment>
+<pinref part="IC1" gate="G$1" pin="CANH"/>
+<pinref part="J1" gate="G$1" pin="2"/>
+<wire x1="142.24" y1="78.74" x2="160.02" y2="78.74" width="0.1524" layer="91"/>
+</segment>
+</net>
+<net name="N$58" class="0">
+<segment>
+<pinref part="J1" gate="G$1" pin="1"/>
+<wire x1="160.02" y1="81.28" x2="157.48" y2="81.28" width="0.1524" layer="91"/>
+<wire x1="157.48" y1="81.28" x2="157.48" y2="83.82" width="0.1524" layer="91"/>
+<pinref part="D12" gate="G$1" pin="A"/>
 </segment>
 </net>
@@
 <text x="-5.08" y="119.38" size="1.27" layer="91">fc=301[Hz]</text>
 <text x="104.14" y="127" size="1.27" layer="91">fc=168.5[kHz]</text>
+<text x="228.6" y="45.72" size="1.778" layer="91">自動放電回路</text>
 </plain>
 <instances>

Commit message: [fix]キッカーボードを25[V]仕様に変更(部品表はまだ)
Parts:
- C1: value 0.33n -> 0.47n
- C6: value 0.22u -> 4.7u
- D1: value SMAJ54A -> SMAJP4KE30A
- L1: value 47u -> 15u; device Passive:L60 -> Passive:L50
- L2: value 5.6u -> 8.2u; device Passive:L8682 -> SRP6060FA-220M:SRP6060FA-220M
- R10: value 100k -> 33k
- R11: value 4.7k -> 3.3k
- R21: value 2.4k -> 3.3k
- R22: value 560 -> 750
- R3: value 13k -> 10k
Connections:
- removed net N$51: IC2.!ACK, R49.1
- new net USBACK: IC2.!ACK, R49.1, U1.PIO0_18/SCT0_OUT5
- net +3V3: now also R49.2
- net +5V: no longer R49.2
Other:
- note added: "->Fsw_nominal=1.25[MHz]"
- note added: "Av=185 ((760+3.3k)/22)"
- note added: "Fsw_max=2.35[MHz]@20[V]"
- note added: "Fsw_max=3.18[MHz]@25[V]"
- note added: "IL_peak=1.67[A]"
- note added: "Imax=6[A]"
- note added: "Io=1.5[A]"
- note added: "Iout_max=0.55[mA]@I=6]A]"
- note added: "Lmin=8.7[uH]@25[V]"
- note added: "Vhys=2.0[V]"
- note added: "Vin_min=20.4[V] Vin_max=25.2[V]"
- note added: "Vout_max=2.21[V]@I=6[A]"
- note added: "Vsense_max=12[mV]@I=6[A]"
- note added: "Vth=19.2[V](3.2[V/cell])"
- note added: "deltaIL=267[mA]@20[V]"
- note added: "deltaIL=347[mA]@25[V]"
- note added: "fc=332[Hz]"
- note added: "fc=83.6[kHz]"
- note removed: "->Fsw_nominal=500[kHz]"
- note removed: "Av=135 ((560+2.4k)/22)"
- note removed: "Fsw_max=1.6[MHz]@50[V]"
- note removed: "Fsw_max=840[kHz]@14[V]"
- note removed: "IL_peak=1.70[A]"
- note removed: "Imax=8[A]"
- note removed: "Iout_max=0.73[mA]@I=8[A]"
- note removed: "Lmin=30[uH]@50[V]"
- note removed: "Vhys=2.6[V]"
- note removed: "Vin_min=14[V] Vin_max=50[V]"
- note removed: "Vout_max=2.15[V]@I=8[A]"
- note removed: "Vsense_max=16[mV]@I=8[A]"
- note removed: "Vth=13.64[V]"
- note removed: "deltaIL=390[mA]@50[V]"
- note removed: "deltaIL=73[mA]@14[V]"
- note removed: "fc=168.5[kHz]"
- note removed: "fc=301[Hz]"
- moved on the sheet: D10, R49

Commit message: [fix]ファイルが壊れてた
Parts:
- removed R15: 10, Passive:R2012
- C1, C11, C12, C13, C14, C16, C17, C18, C19, C2, C20, C22, C3, C4, C7: device Passive:C1608 -> MotorDriver:C1005
- C10, C9: device Passive:C2012 -> MotorDriver:C1005
- C15: value (none) -> 0.1u; device Passive:C1608 -> MotorDriver:C1005
- C21: device Passive:C3216 -> MotorDriver:C3216
- C23, C24: value (none) -> 10p; device MotorDriver:C1608 -> MotorDriver:C1005
- C6: device Passive:C1608 -> MotorDriver:C1608
- C8: device Passive:C3216 -> MotorDriver:C1608
- D1, D4: device Diode:ZENER-DO-214AC -> MotorDriver:SBD-DO-214AC
- D10, D7, D8, D9: device Diode:SBD-SOD523 -> MotorDriver:SBD-SOD523
- D12: device MotorDriver:MOTORDRIVER_SBD-SOD523 -> MotorDriver:SBD-SOD523
- LED4, LED5: device Opto:LED1608 -> MotorDriver:LED1608
- R1, R10, R11, R16, R17, R18, R2, R20, R21, R22, R23, R26, R27, R29, R3, R30, R31, R32, R33, R35, R37, R38, R39, R40, R41, R5, R50, R6, R8, R9: device Passive:R1608 -> MotorDriver:R1005
- R13, R14, R34, R4, R7: device Passive:R1608 -> MotorDriver:R1608
- R42: value 220 -> 330; device Passive:R1608 -> MotorDriver:R1005
- R43, R44: device MotorDriver:R1608 -> MotorDriver:R1005
- R45, R46, R47: value 100 -> 330; device MotorDriver:R1608 -> MotorDriver:R1005
- U1: device MotorDriver_Rev1:LPC1549JBD48_LPC1549JBD48 -> MotorDriver:LPC1549JBD48
Connections:
- removed net N$23: R15.2, U$2.S
- net GND: now also U$2.S; no longer R15.1
