File: KickerBoard/KickerBoard.sch (EAGLE design)
At the start: 125 parts, among them IC1 MAX3051ESA+, IC2 TPD4S014DSQR, J1 SM03B-ZESS-TB, J2 J_USB_MICROAB_HIROSE_ZX62-AB-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, Q1 TK12P60W, Q4 BSS138, Q5 BSP130, Q6 ZXTN08400BFF, U1 LPC1549JBD48, U10 AD8601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

Commit message: tmpからもってきた
Parts:
- added R15: 2.2k, Passive:R1608
- C16, C20: value 1u -> 0.1u
- C5: value 22u -> 220u
- D3: device Diode:DIODE-DO-214AB -> diode:DIODE-DO-214AB
- D5, D6: device Diode:DIODE-SMPC -> diode:DIODE-SMPC
- JP1, JP2: device con-Molex:5569-02A2 -> con-molex:5569-02A2
- Q1: device Transistor:MOS-N-DPAK -> transistor:MOS-N-DPAK
- Q4: device Transistor:MOS-N-SOT23 -> transistor:MOS-N-SOT23
- Q5: device Transistor:MOS-N-SOT223 -> transistor:MOS-N-SOT223
- R2: value 240k -> 120k
Connections:
- removed net ID: IC2.ID, J2G$2.ID, U1.PIO0_13/ADC1_6
- new net N$23: IC2.!EN, R15.2
- net GND: now also R15.1; no longer IC2.!EN
Other:
- note added: "->Fsw_nominal=1.00[MHz]"
- note added: "IL_peak=1.71[A]"
- note added: "Lmin=10[uH]@25[V]"
- note added: "Vhys=3.0[V]"
- note added: "Vth=19.8[V](3.3[V/cell])"
- note added: "deltaIL=320[mA]@20[V]"
- note added: "deltaIL=416[mA]@25[V]"
- note removed: "->Fsw_nominal=1.25[MHz]"
- note removed: "IL_peak=1.67[A]"
- note removed: "Lmin=8.7[uH]@25[V]"
- note removed: "Vhys=2.0[V]"
- note removed: "Vth=19.2[V](3.2[V/cell])"
- note removed: "deltaIL=267[mA]@20[V]"
- note removed: "deltaIL=347[mA]@25[V]"
