File: KickerBoard/KickerBoard.brd (EAGLE design)
At the start: 75 x 50 mm, 125 parts, among them IC1 MAX3051ESA+, IC2 TPD4S014DSQR, J1 SM03B-ZESS-TB, J2 J_USB_MICROAB_HIROSE_ZX62-AB-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, Q1 TK12P60W, Q4 BSS138, Q5 BSP130, Q6 ZXTN08400BFF, U1 LPC1549JBD48, U10 AD8601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

Commit message: tmpからもってきた
Parts:
- added R15: 2.2k, Passive:1608
- C16, C20: value 1u -> 0.1u
- C5: value 22u -> 220u
- D3: device Diode:DO-214AB -> diode:DO-214AB
- D5, D6: device Diode:SMPC -> diode:SMPC
- JP1, JP2: device con-Molex:5569-02A2 -> con-molex:5569-02A2
- Q1: device Transistor:DPAK-3 -> transistor:DPAK-3
- Q4: device Transistor:SOT23-3 -> transistor:SOT23-3
- Q5: device Transistor:SOT223 -> transistor:SOT223
- R2: value 240k -> 120k
Connections:
- removed net ID: IC2.5, J2.P$4, U1.21
- new net N$23: IC2.3, R15.2
- net GND: now also R15.1; no longer IC2.3
Routing:
- net ID: track 11.5 -> 0.00 mm, vias 1 -> 0
- net N$23: track 0.00 -> 2.87 mm
- net GND: track 43.9 -> 41.4 mm
