File: MainBoard/MainBoard.brd (EAGLE design)
At the start: 75 x 50 mm, 83 parts, among them CN9 UX60SC-MB-5ST, J1 53375-0610, J2 53375-0610, J3 53375-0610, J4 53375-0610, J5 53375-0610, J6 53375-0610, U1 MCP1700T-33, U2 ADR5041, U3 FT232RL, U4 LM5160QPWPRQ1, U5 LPC1549JBD48

Commit message: tmpからもってきた
Parts:
- removed C15: 0.1u, MotorDriver:C1608
- removed C4, C5: 22u, MotorDriver:C1608
- removed C6: 10u, MotorDriver:C1608
- removed CN7: (no value), Connector:T-CON
- removed CN9: UX60SC-MB-5ST, con-Hirose:UX60SC-MB-5ST
- removed D1: (no value), MotorDriver:DO-214AC
- removed L1: 22u, Passive:L4040
- removed LED10, LED2, LED3, LED4, LED5, LED6, LED7, LED8: (no value), MotorDriver:LED1608
- removed R17, R18, R19, R20: 220, MotorDriver:R1608
- removed R21: (no value), MotorDriver:R1608
- removed SW2: (no value), MotorDriver:SKRP
- removed U3: FT232RL, ic-FTDI:SSOP28
- added CBP1, CBP2: 10u, MotorDriver:C1608
- added CBST: 22n, MotorDriver:C1608
- added COUT1, COUT2: 22u, MotorDriver:C1608
- added COUT3, COUT4, COUT5: 0.1u, MotorDriver:C1608
- added D5: MBR230LSFT1G, MBR230LSFT1G:SODFL3616X98N
- added GND: UX60SC-MB-5ST, con-Hirose:UX60SC-MB-5ST
- added IC1: ESP-WROOM-02, esp-wroom-02:ESP-WROOM-02
- added IC2: TS30042-M033QFNR, TS30042-M033QFNR:QFN50P300X300X100-17N
- added IC3: MAX33053EASA+, MAX33053EASA+:SOIC127P605X145-8N
- added L2: SLF7045T-220MR90-PF, SLF7045T-220MR90-PF:INDPM7070X480N
- added Q1, Q2, Q3: NP52N06SLG-E2-AY, NP52N06SLG-E2-AY:NP52N06SLGE2AY
- added RBOT: 3k, MotorDriver:R1608
- added RPLP: 10k, MotorDriver:R1608
- added RTOP: 8k, MotorDriver:R1608
- added U6: ESP-WROOM-32, esp32:ESP-WROOM-32
- added U7, U8: TLP185(GR,E(O, TLP185(GR_E(O:SOP254P700X220-4N
- added Y1: CSTCE12M0G55-R0, CSTCE12M0G55-R0:CSTCE12M0G55-R0
- C1: value 10n -> 0.1u
- C2: value 22n -> 33p
- C3: value 1u -> 33p
- F1: value 15 -> 20
- F2: value 10 -> 20
- J1, J2, J3, J4, J5, J6: value 53375-0610 -> 53375-0310; device MotorDriver:53375-0610 -> 53375-0310:53375-0310
- R1: value 91k -> 1k
- R13, R14: value 220 -> 1k
- R15, R16: value 220 -> 120
- R2: value 130k -> 1k
- R3: value 13k -> 1k
- R4: value 10 -> 1k
- R5: value 3.3k -> 1k
- R6: value 2.2k -> 1k
- R7: value 1 -> 1k
- U4: value LM5160QPWPRQ1 -> TLP185(GR,E(O; device LM5160QPWPRQ1:SOP65P640X110-15N -> TLP185(GR_E(O:SOP254P700X220-4N
- moved R16 66.6 mm to (6.48, 24.3), turned to 90 degrees
- moved R14 57.8 mm to (17.5, 40.0), flipped to the top, turned to 0 degrees
- moved C2 49.3 mm to (68.0, 29.4), turned to 270 degrees
- moved C3 45.3 mm to (68.0, 26.4), turned to 90 degrees
- moved R7 41.1 mm to (17.5, 42.9), flipped to the top, turned to 180 degrees
- moved R3 41.0 mm to (38.5, 39.9), flipped to the top, turned to 0 degrees
- moved R1 40.1 mm to (38.5, 42.9), flipped to the top, turned to 0 degrees
- moved R2 39.5 mm to (38.5, 41.4), flipped to the top, turned to 0 degrees
- moved U4 39.2 mm to (38.5, 41.4), turned to 90 degrees
- moved R4 38.0 mm to (28.0, 42.9), flipped to the top, turned to 180 degrees
- moved R11 33.6 mm to (17.5, 41.4), flipped to the top
- moved R5 31.0 mm to (28.0, 41.4), flipped to the top, turned to 0 degrees
- moved R6 29.5 mm to (28.0, 39.9), flipped to the top
- moved CN1 29.2 mm to (71.1, 31.3)
- moved C1 23.1 mm to (53.3, 1.97), flipped to the top, turned to 270 degrees
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Connections:
- removed net !CS1: J1.2, U5.2
- removed net !CS2: J2.2, U5.3
- removed net !CS3: J3.2, U5.6
- removed net !CS4: J4.2, U5.8
- removed net !CS5: J5.2, U5.9
- removed net !CS6: J6.2, U5.12
- removed net !ISP: C15.1, R21.1, SW2.B1, SW2.B2, U5.24, U5.5
- removed net CLK: J1.5, J2.5, J3.5, J4.5, J5.5, J6.5
- removed net LED1: LED1.A, U5.21
- removed net LED2: LED2.A, U5.28
- removed net LED3: LED3.A, U5.29
- removed net LED4: LED4.A, U5.33
- removed net LED5: LED5.A, U5.35
- removed net LED6: LED6.A, U5.36
- removed net LED7: LED7.A, U5.43
- removed net LED8: LED8.A, U5.44
- removed net MISO: J1.3, J2.3, J3.3, J4.3, J5.3, J6.3, U5.7
- removed net MOSI: J1.4, J2.4, J3.4, J4.4, J5.4, J6.4, U5.4
- removed net N$11: C4.2, D1.A, L1.2, LED10.A, R5.2, R7.2
- removed net N$12: U3.17, U3.4
- removed net N$14: CN9.2, U3.16
- removed net N$15: CN9.3, U3.15
- removed net N$20 (its old number): LED3.K, R15.2
- removed net N$29: LED4.K, R16.2
- removed net N$30: LED2.K, R14.2
- removed net N$4: C1.1, L1.1, R4.1, U4.12, U4.13
- removed net VMOTOR1: CN2.P, CN3.P, CN4.P, F1.2
- removed net VMOTOR2: CN5.P, CN6.P, F2.2
- new net !MCLP: J1.1, J2.1, J3.1, J4.1, J5.1, J6.1, U5.2
- new net +3.3V: IC3.5
- new net 3.3V: U5.3
- new net CAN0_RD: IC3.4, U5.21
- new net CAN0_TD: IC3.1, U5.13
- new net CANH: IC3.7, J1.2, J2.2, J3.2, J4.2, J5.2, J6.2, R15.2, R16.1
- new net CANL: IC3.6, J1.3, J2.3, J3.3, J4.3, J5.3, J6.3, R15.1, R16.2
- new net D+: GND.3, U5.35
- new net D-: GND.2, U5.36
- new net KICKER: CN6.P, F2.2
- new net LSW1: U4.1, U5.7
- new net LSW2: U5.8, U7.1
- new net LSW3: U5.9, U8.1
- new net N$16: CBST.1, D5.1, IC2.1, IC2.12, IC2.13, IC2.17, L2.1
- new net N$17: C2.1, U5.32, Y1.1
- new net N$22: IC2.8, RPLP.2, RTOP.2
- new net N$23: C1.1, IC3.3
- new net N$25: R14.1, U8.2
- new net N$28: COUT4.1, Q3.1, R11.1, R7.2
- new net STBY: IC3.8, U5.4
- new net VMOTOR: CN2.P, CN3.P, CN4.P, CN5.P, F1.2, U4.4, U7.4, U8.4
- net +3V3: now also IC1.1, U6.2; no longer R21.2
- net +5V: now also COUT1.1, COUT2.1, L2.2, LED1.A, RPLP.1, RTOP.1; no longer D1.K, J1.1, J2.1, J3.1, J4.1, J5.1, J6.1
- net GND: now also C1.2, CBP1.2, CBP2.2, COUT1.2, COUT2.2, COUT3.2, COUT4.2, COUT5.2, D5.2, GND.5, GND.S1, GND.S2, IC1.13, IC1.18, IC1.19, IC1.8, IC1.9, IC2.14, IC2.16, IC2.4, IC3.2, Q1.2, Q2.2, Q3.2, R11.2, R14.2, R2.2, R3.2, R5.2, R6.2, RBOT.2, U6.1, U6.15, U6.38, U6.GND, Y1.2; no longer C15.2, C6.2, CN2.N, CN3.N, CN4.N, CN7.N, CN9.5, CN9.S1, CN9.S2, J1.6, J2.6, J3.6, J4.6, J5.6, J6.6, R11.1, R14.1, R15.1, R16.1, R17.1, R18.1, R19.1, R20.1, R3.1, R6.1, SW2.A1, SW2.A2, U3.18, U3.21, U3.25, U3.26, U3.7, U4.1, U4.15, U4.2
- net N$1: now also CN2.N, Q1.3; no longer R1.2, U4.5
- net N$13: now also GND.1; no longer CN9.1, U3.20
- net N$19: now also COUT3.1, Q2.1, R4.2, R5.1; no longer LED10.K, R11.2
- net N$2: now also R1.2, U4.3; no longer R2.1, R3.2, U4.4
- net N$21: now also IC2.5, RBOT.1; no longer LED5.K, R17.2
- net N$24: now also CBST.2, IC2.10; no longer LED6.K, R18.2
- net N$26: now also R7.1, U8.3; no longer LED7.K, R19.2
- net N$27: now also C3.1, U5.31, Y1.3; no longer LED8.K, R20.2
- net N$3: now also COUT5.1, Q1.1, R1.1, R2.1; no longer C6.1, R7.1
- net N$5: now also CN3.N, Q2.3; no longer C1.2, U4.11
- net N$6: now also R3.1, U4.2; no longer C3.1, U4.10, U4.8
- net N$7: now also R6.1, U7.2; no longer C2.1, U4.6
- net N$8: now also R4.1, U7.3; no longer C5.2, R5.1, R6.2, U4.9
- net N$9: now also CN4.N, Q3.3; no longer C4.1, C5.1, R4.2
- net RX: no longer U3.1
- net TX: no longer U3.5
- net V+: now also CBP1.1, CBP2.1, IC2.11, IC2.2, IC2.3; no longer CN7.P, R1.1, R2.2, U4.3
- net XBEE_RX: now also IC1.11, U6.35
- net XBEE_TX: now also IC1.12, U6.34
Routing:
- net V+: track 0.00 -> 83.2 mm, vias 47 -> 57
- net CANH: track 0.00 -> 64.4 mm
- net CANL: track 0.00 -> 63.5 mm, vias 0 -> 2
- net !CS1: track 60.9 -> 0.00 mm
- net +5V: track 120.5 -> 175.9 mm, vias 1 -> 4
- net !MCLP: track 0.00 -> 53.2 mm, vias 0 -> 2
- net +3V3: track 112.1 -> 162.8 mm, vias 5 -> 3
- net LSW3: track 0.00 -> 50.2 mm, vias 0 -> 1
- net MOSI: track 48.4 -> 0.00 mm
- net MISO: track 48.0 -> 0.00 mm
- net LSW2: track 0.00 -> 45.2 mm, vias 0 -> 1
- net !CS2: track 43.7 -> 0.00 mm, vias 1 -> 0
- net D-: track 0.00 -> 41.8 mm
- net CLK: track 38.1 -> 0.00 mm
- net !CS3: track 34.6 -> 0.00 mm
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- added copper zone on layer 1, net KICKER
- added copper zone on layer 16, net KICKER
- added copper zone on layer 16, net N$1
- added copper zone on layer 16, net N$5
- added copper zone on layer 16, net N$9
- added copper zone on layer 1, net VMOTOR
- added copper zone on layer 16, net VMOTOR
- removed copper zone on layer 16, net N$11
- removed copper zone on layer 1, net N$13
- removed copper zone on layer 16, net N$4
- removed copper zone on layer 1, net VMOTOR1
- removed copper zone on layer 16, net VMOTOR1
- removed copper zone on layer 1, net VMOTOR2
- removed copper zone on layer 16, net VMOTOR2
